File: hardware/can_node_board_hw/can_node_board_pwr.sch (KiCad schematic (older format))
At the start: 0 parts

Commit message: Completed the schematic for the PIC18F4620 SPI Test. I will note that the KiCAD DRC on the schematic still gives --Pin connected to other pins, but not driven by any pin-- warnings, and I have not been able to clear those...
Parts:
- added R?: R, symbol Device:R
Changed lines of the file:
@@
 Comment4 "Author: Abdullah Almosalami"
 $EndDescr
+$Comp
+L Device:R R?
+U 1 1 6184B4BE
+P 5100 3300
+F 0 "R?" H 5170 3346 50  0000 L CNN
+F 1 "R" H 5170 3255 50  0000 L CNN
+F 2 "" V 5030 3300 50  0001 C CNN
+F 3 "~" H 5100 3300 50  0001 C CNN
+	1    5100 3300
+	1    0    0    -1
+$EndComp
 $EndSCHEMATC
